Commit message: Added working sonar to tbot.

File: src/tbot_description/urdf/tbot.xacro (robot description, xacro)
@@ -1,7 +1,7 @@
 <?xml version='1.0'?>
 <robot name="tablebot" xmlns:xacro="http://www.ros.org/wiki/xacro">
-  <xacro:include filename="$(find tbot_description)/urdf/tbot.gazebo" />
-  <xacro:include filename="$(find tbot_description)/urdf/materials.xacro" />
-  <xacro:include filename="$(find tbot_description)/urdf/macros.xacro" />
+  <!-- xacro:include filename="$(find tbot_description)/urdf/tbot.gazebo" / -->
+  <!--<xacro:include filename="$(find tbot_description)/urdf/materials.xacro" / -->
+	  <!-- <xacro:include filename="$(find tbot_description)/urdf/macros.xacro" / -->
   <link name='chassis'>
     <pose>0 0 0.1 0 0 0</pose>
@@ -139,3 +139,95 @@
     <joint_properties damping="0.0" friction="0.0"/>
   </joint>
+  <joint name="sonar_joint" type="fixed">
+	  <axis xyz="0 1 0" />
+	  <origin xyz=".25 0 0" rpy="0 0 0" />
+	  <parent link="chassis" />
+	  <child link="sonar" />
+  </joint>
+<!--Sonar link -->
+<link name="sonar">
+    <pose>0 0 0 0 0 0</pose>
+    <inertial>
+      <mass value="1.0"/>
+      <origin xyz="0 0 0" rpy=" 0 0 0"/>
+      <inertia
+          ixx="0.5" ixy="0" ixz="0"
+          iyy="1.0" iyz="0"
+          izz="0.1"
+      />
+    </inertial>
+	<!--
+    <collision name="sonar_collision">
+      <geometry>
+        <box size=".1 .1 .1"/>
+      </geometry>
+    </collision>
+	-->
+    <visual name="sonar_visual">
+      <origin xyz="0 0 0" rpy=" 0 0 0"/>
+      <geometry>
+        <box size=".05 .1 .1"/>
+      </geometry>
+    </visual>
+</link>
+<!-- Gazebo chassis color -->
+<gazebo reference="chassis">
+  <material>Gazebo/Orange</material>
+</gazebo>
+<!-- Diff Drive Gazebo Plugin -->
+<gazebo>
+	<plugin name="differential_drive_controller" filename="libgazebo_ros_diff_drive.so">
+	  <legacyMode>false</legacyMode>
+	  <alwaysOn>true</alwaysOn>
+	  <updateRate>20</updateRate>
+	  <leftJoint>left_wheel_hinge</leftJoint>
+	  <rightJoint>right_wheel_hinge</rightJoint>
+	  <wheelSeparation>0.3</wheelSeparation>
+	  <wheelDiameter>0.2</wheelDiameter>
+	  <torque>20</torque>
+	  <commandTopic>cmd_vel</commandTopic>
+	  <odometryTopic>odom</odometryTopic>
+	  <odometryFrame>odom</odometryFrame>
+	  <robotBaseFrame>chassis</robotBaseFrame>
+	</plugin>
+</gazebo>
+<!-- Sonar Gazebo Plugin -->
+<gazebo reference="sonar">
+    <material>Gazebo/Green</material>
+    <sensor type="ray" name="sonar_sensor">
+        <pose>0 0 0 0 0 0</pose>
+        <update_rate>5</update_rate>
+        <ray>
+            <scan>
+                <horizontal>
+                    <samples>5</samples>
+                    <resolution>1.0</resolution>
+                    <min_angle>-0.25</min_angle>
+                    <max_angle>0.25</max_angle>
+                </horizontal>
+                <vertical>
+                    <samples>5</samples>
+                    <resolution>1</resolution>
+                    <min_angle>-0.25</min_angle>
+                    <max_angle>0.25</max_angle>
+                </vertical>
+            </scan>
+            <range>
+                <min>0.01</min>
+                <max>0.75</max>
+                <resolution>0.01</resolution>
+            </range>
+        </ray>
+        <plugin filename="libgazebo_ros_range.so" name="gazebo_ros_range">
+            <!--<gaussianNoise>0.005</gaussianNoise> -->
+            <gaussianNoise>0.0</gaussianNoise>
+            <alwaysOn>true</alwaysOn>
+            <updateRate>5</updateRate>
+            <topicName>sonar1</topicName>
+            <frameName>sonar</frameName>
+            <fov>0.5</fov>
+            <radiation>ultrasound</radiation>
+        </plugin>
+    </sensor>
+</gazebo>
 </robot>

Commit message: Put sonar at 45 degree angle.

File: src/tbot_description/urdf/tbot.xacro (robot description, xacro)
@@ -141,5 +141,5 @@
   <joint name="sonar_joint" type="fixed">
 	  <axis xyz="0 1 0" />
-	  <origin xyz=".25 0 0" rpy="0 0 0" />
+	  <origin xyz=".25 0 0" rpy="0 0.7854 0" />
 	  <parent link="chassis" />
 	  <child link="sonar" />
@@ -150,5 +150,5 @@
     <inertial>
       <mass value="1.0"/>
-      <origin xyz="0 0 0" rpy=" 0 0 0"/>
+      <origin xyz="0 0 0" rpy="0 0 0"/>
       <inertia
           ixx="0.5" ixy="0" ixz="0"
